Commit message: Add SCARA_with_noise_example
Add SCARA_with_noise_example

File: Matlab/urdf/scara/scara_noisy.urdf (robot description, URDF)
Before this commit: robot scara, 7 links, 6 joints
Joints:
- joint joint0: origin xyz=0 0 0.375 rpy=0 0 0 -> xyz=0.0 0.0 0.375 rpy=0 0 0
- joint joint1: origin xyz=0 0.5 0.025 rpy=0 0 0 -> xyz=0.01 0.51 -0.024 rpy=0.0175 0.0175 -0.0175
- joint joint2: origin xyz=0.5 0.0 0.0 rpy=0 0 0 -> xyz=0.51 -0.01 0.01 rpy=0.0175 -0.0175 0.0175
- joint joint3: origin xyz=0.0 0.0 -0.25 rpy=0 0 0 -> xyz=-0.01 -0.01 -0.29 rpy=-0.0175 -0.0175 -0.0175
